File: layouts/dev/dev.kicad_pcb (KiCad board)
At the start: 4 copper layers, 32.5 x 59.6 mm, 73 parts

Commit message: feat: SWD on a proper ARM Cortex Debug connector
Samtec SHF-105-01-L-D-RA, right-angle, keyed shroud, 2x5 at 1.27 mm. The
J-Link EDU Mini cable plugs straight in, and so does ST-LINK V2/V3 - it is
a standard rather than somebody's pin order. Right-angle because a vertical
one with the cable attached stands about 7 mm above the laminate, exactly
where a probe and fingers need to be during bring-up.

Two grounds sit between the fast lines (pin 3 between SWDIO and SWCLK,
pin 5 between SWCLK and SWO), so each has a return in the neighbouring
ribbon wire. That matters most for SWO, which carries the ITM console.

The four positions on the left header that used to carry SWD (5 NRST,
6 SWDIO, 8 SWCLK, 9 SWO) are left WITHOUT A NET. They were not reassigned
and not removed: the header keeps twelve positions and the same footprint,
four of them simply unconnected. A header is where a person plugs a wire
without reading the docs, so the same shape must not mean different things
in two revisions.

Placement, routing and the outline are untouched: 95 segments and 15 vias
before and after, no footprint moved, CN1 is the only addition.

Co-Authored-By: Claude Opus 5 (1M context) <noreply@anthropic.com>
Claude-Session: https://claude.ai/code/session_01BM8NndJbzBEDPtrpVjN835
Parts:
- added CN1: , Samtec_SHF_105_01_L_D_RA:CONN-THT_10P-P1.27_SHF-105-01-L-D-RA, F.Cu at (0.00, 0.00)
Connections:
- J2 pad 5: NRST -> 5
- J2 pad 6: SWDIO -> 6
- J2 pad 8: SWCLK -> 8
- J2 pad 9: SWO -> 9
Other:
- outline, holes or cut-outs redrawn

Commit message: chore: board file after the SWD rebuild
ato build plus board_setup.py, no source change. Picks up CN1 in the PCB
and the net classes rewritten in the project file.

Co-Authored-By: Claude Opus 5 (1M context) <noreply@anthropic.com>
Claude-Session: https://claude.ai/code/session_01BM8NndJbzBEDPtrpVjN835
Parts:
- moved CN1 52.8 mm to (15.4, 50.5), turned to 90 degrees
- moved C8 26.4 mm to (15.2, 7.62)
- moved R12 16.8 mm to (50.0, 17.0)
- moved R13 16.8 mm to (50.0, 15.5)
- moved C5 6.51 mm to (32.8, 17.8), turned to 0 degrees
- moved C6 4.10 mm to (32.8, 16.0)
- moved C10 4.07 mm to (27.7, 30.0)
- moved C18 4.07 mm to (27.7, 28.4)
- moved R17 4.03 mm to (27.7, 32.3)
- moved C7 3.81 mm to (31.0, 11.9), turned to 90 degrees
- moved R2 3.49 mm to (28.4, 16.0), turned to 90 degrees
- moved R1 2.79 mm to (34.0, 11.9)
- moved X2 2.29 mm to (30.2, 16.5), turned to 90 degrees
- moved R7 2.17 mm to (34.8, 40.4), turned to 0 degrees
- moved C3 1.57 mm to (23.9, 9.40)
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Routing:
- net SWDIO: track 0.00 -> 38.2 mm, vias 0 -> 1
- net SWCLK: track 0.00 -> 36.8 mm, vias 0 -> 1
- net +3V3: track 14.6 -> 35.1 mm, vias 1 -> 5
- net GND: track 11.6 -> 31.3 mm, vias 10 -> 22
- net NRST: track 0.00 -> 12.0 mm
- net BOOT0: track 0.00 -> 12.0 mm, vias 0 -> 2
- net PMIC_SDA: track 0.00 -> 10.4 mm, vias 0 -> 1
- net PB5: track 0.00 -> 9.52 mm
- net PMIC_SCL: track 0.00 -> 8.57 mm, vias 0 -> 1
- net 27: track 0.00 -> 7.02 mm, vias 0 -> 1
- net 26: track 0.00 -> 5.40 mm, vias 0 -> 1
- net CHG_INT: track 0.00 -> 5.22 mm, vias 0 -> 1
- net VLXSMPS: track 0.00 -> 5.20 mm
- net VFBSMPS: track 0.00 -> 4.28 mm
- net PB7: track 0.00 -> 3.69 mm, vias 0 -> 1
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Other:
- outline, holes or cut-outs redrawn

Commit message: feat: stitch the thermal pads of the leadless packages to ground
For the STM32WB55 in UFQFPN-48 this is not a nicety: that package has no
VSS pin at all, so the pad under the body is the chip's ONLY connection to
ground, and the In1 plane sits 0.2104 mm below the top layer with no other
way down. U1 gets 5x5 = 25 vias in its 5.50 mm pad at a 1.12 mm pitch,
U4 gets 2x2 in its 2.70 mm pad. Vias are 0.50/0.25, 0.25 mm of pad left
around each.

Packages are matched by footprint name (QFN/SON/DFN), the way sieci_bga
already matches BGA - designators renumber on every rebuild, package names
do not. A pad-area threshold separates thermal pads from signal ones.

The grid follows placement: it is recomputed from the pad position and
orientation on every run, and the previous one is deleted first, so moving
or rotating a part carries it along and ato build cannot lose it.

Two findings while doing this, both inherited from gps_tracker-6l and both
reported by the script instead of silently drilled:

* TPS63020DSJR and BQ27441 have NO real thermal pad in their footprints -
  a 0.01 x 0.01 mm placeholder sits where the exposed pad belongs. Both
  datasheets require that pad on PGND/VSS. Left alone for now; the script
  names them on every run.
* These vias sit in a pad and must be resin filled. The 0.25 mm drill is
  in the range JLCPCB fills, but on four layers that is a paid option.

Routing untouched: 280 segments and the 56 routing vias before and after.

Co-Authored-By: Claude Opus 5 (1M context) <noreply@anthropic.com>
Claude-Session: https://claude.ai/code/session_01BM8NndJbzBEDPtrpVjN835
Routing:
- net GND: vias 22 -> 51
Other:
- outline, holes or cut-outs redrawn
